File: kicad/_autosave-dac.kicad_pcb (KiCad board)
At the start: 4 copper layers, 54.5 x 61.2 mm, 87 parts, among them J1 I2S, J2 I2S, J3 ANALOG PWR, J4 5V, J5 AUDIO OUT, U1 ES9039Q2M, U2 OPA1612AxD, U3 OPA1612AxD, U4 LT3046ATC+, U5 TPS7A39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

Commit message: Added images and small PCB changes
Routing:
- net /+15V: track 17.2 -> 20.0 mm, vias 0 -> 1
- net /-15V: track 16.5 -> 16.3 mm, vias 0 -> 1
- net GND: track 32.6 -> 32.5 mm, vias 201 -> 202
