File: kicad/dac.kicad_sch (KiCad schematic)
At the start: 42 parts, among them J1 I2S, J2 I2S, J3 ANALOG PWR, J4 5V, U1 ES9039Q2M, U4 LT3046ATC+, U5 TPS7A39, Y1 CE3391-49.152

Commit message: V1.0
Parts:
- C3, C32, C7: Vendor Murata -> Kyocera
- R8, R9: now in the parts list
Connections:
- net +15V: now also J3.3 (Pin_3); no longer J3.1 (Pin_1)
- net -15V: now also J3.1 (Pin_1); no longer J3.3 (Pin_3)
Changed lines of the file:
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@@
 			)
 		)
-		(property "Description" "GRM02YD70E104ME01L"
+		(property "Description" "KGM05AR71C104KN"
 			(at 106.68 85.09 0)
 			(effects
@@
 			)
 		)
-		(property "Vendor" "Murata"
+		(property "Vendor" "Kyocera"
 			(at 106.68 85.09 0)
 			(effects
@@
 			)
 		)
-		(property "Description" "GRM02YD70E104ME01L"
+		(property "Description" "KGM05AR71C104KN"
 			(at 130.81 111.76 0)
 			(effects
@@
 			)
 		)
-		(property "Vendor" "Murata"
+		(property "Vendor" "Kyocera"
 			(at 130.81 111.76 0)
 			(effects
@@
 		(unit 1)
 		(exclude_from_sim no)
-		(in_bom no)
+		(in_bom yes)
 		(on_board yes)
 		(dnp no)
@@
 			)
 		)
-		(property "Description" "ERA-1AEB472C"
+		(property "Description" "ERA-3AEB472V"
 			(at 173.99 116.84 0)
 			(effects
@@
 		(unit 1)
 		(exclude_from_sim no)
-		(in_bom no)
+		(in_bom yes)
 		(on_board yes)
 		(dnp no)
@@
 			)
 		)
-		(property "Description" "ERA-1AEB472C"
+		(property "Description" "ERA-3AEB472V"
 			(at 166.37 116.84 0)
 			(effects
@@
 			)
 		)
-		(property "Description" "GRM02YD70E104ME01L"
+		(property "Description" "KGM05AR71C104KN"
 			(at 114.3 106.68 0)
 			(effects
@@
 			)
 		)
-		(property "Vendor" "Murata"
+		(property "Vendor" "Kyocera"
 			(at 114.3 106.68 0)
 			(effects
@@
 		(lib_id "Connector:Conn_01x03_Pin")
 		(at 25.4 38.1 0)
+		(mirror x)
 		(unit 1)
 		(exclude_from_sim no)
@@
 		(dnp no)
 		(property "Reference" "J3"
-			(at 22.86 37.846 90)
+			(at 22.86 38.354 90)
 			(effects
 				(font
