File: kicad/output.kicad_sch (KiCad schematic)
At the start: 37 parts, among them J5 AUDIO OUT, U2 OPA1612AxD, U3 OPA1612AxD

Commit message: V1.0
Parts:
- R15, R16, R22, R23: now in the parts list
Changed lines of the file:
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@@
 		(unit 1)
 		(exclude_from_sim no)
-		(in_bom no)
+		(in_bom yes)
 		(on_board yes)
 		(dnp no)
@@
 			)
 		)
-		(property "Description" "ERA-1AEB472C"
+		(property "Description" "ERA-3AEB472V"
 			(at 224.79 93.98 0)
 			(effects
@@
 		(unit 1)
 		(exclude_from_sim no)
-		(in_bom no)
+		(in_bom yes)
 		(on_board yes)
 		(dnp no)
@@
 			)
 		)
-		(property "Description" "ERA-1AEB472C"
+		(property "Description" "ERA-3AEB472V"
 			(at 224.79 67.31 0)
 			(effects
@@
 		(unit 1)
 		(exclude_from_sim no)
-		(in_bom no)
+		(in_bom yes)
 		(on_board yes)
 		(dnp no)
@@
 			)
 		)
-		(property "Description" "ERA-1AEB472C"
+		(property "Description" "ERA-3AEB472V"
 			(at 96.52 67.31 0)
 			(effects
@@
 		(unit 1)
 		(exclude_from_sim no)
-		(in_bom no)
+		(in_bom yes)
 		(on_board yes)
 		(dnp no)
@@
 			)
 		)
-		(property "Description" "ERA-1AEB472C"
+		(property "Description" "ERA-3AEB472V"
 			(at 96.52 93.98 0)
 			(effects
